File: PCB/KiCAD/ESP32.kicad_sch (KiCad schematic)
At the start: 27 parts, among them IC1 ESP32-S3-WROOM-1, J2 AFC07-S24ECA-00, J2 AVR-ISP-6, Q1 MMBT5551LT1G, Q2 MMBT5551LT1G, SW1 C255812, SW2 C255812

Commit message: Initial PCB draft
Parts:
- removed C17: ${ALTIUM_VALUE}, CAP 1206_3216 - 0.8MM, symbol ESP32-altium-import:root_2_Capacitor
- removed C23: ${ALTIUM_VALUE}, CAP 1206_3216 - 0.8MM, symbol ESP32-altium-import:root_1_Capacitor
- removed C24: ${ALTIUM_VALUE}, CAP 0603_1608, symbol ESP32-altium-import:root_3_Capacitor
- removed IC1: ESP32-S3-WROOM-1, C:_Users_Henry_Documents_AltiumLL_SamacSys.PcbLib_ESP32S3WROOM1, symbol ESP32-altium-import:root_0_ESP32-S3-WROOM-1
- removed J2: AVR-ISP-6, symbol Connector:AVR-ISP-6
- removed J2: AFC07-S24ECA-00, MOLX-52437-2471, symbol ESP32-altium-import:root_3_mirrored_MOLX-52437-2471
- removed Q1: MMBT5551LT1G, ONSC-SOT-23-3-318-08_V, symbol ESP32-altium-import:root_0_ONSC-NPN-B1E2C3-3
- removed Q2: MMBT5551LT1G, ONSC-SOT-23-3-318-08_V, symbol ESP32-altium-import:root_2_mirrored_ONSC-NPN-B1E2C3-3
- removed R12, R14: ${ALTIUM_VALUE}, RES 0603_1608, symbol ESP32-altium-import:root_2_mirrored_Resistor
- removed R13, R15, R16: ${ALTIUM_VALUE}, RES 0603_1608, symbol ESP32-altium-import:root_0_Resistor
- removed R17, R18, R19: ${ALTIUM_VALUE}, RES 0603_1608, symbol ESP32-altium-import:root_0_mirrored_Resistor
- removed R7: ${ALTIUM_VALUE}, RES 0603_1608, symbol ESP32-altium-import:root_3_Resistor
- added C10: 10uF, Capacitor_SMD:C_1206_3216Metric, symbol Device:C_Small
- added C11, C8: 1uF, Capacitor_SMD:C_0603_1608Metric, symbol Device:C_Small
- added C9: 10pF, Capacitor_SMD:C_0603_1608Metric, symbol Device:C_Small
- added DSP1: ~, Footprints:HS12864G19C Display, symbol PartLibrary:HS12864G19A_Mech
- added H1, H2, H3, H4: MountingHole, MountingHole:MountingHole_3.2mm_M3, symbol Mechanical:MountingHole
- added J1: Conn_01x06, Connector_PinHeader_2.54mm:PinHeader_1x06_P2.54mm_Vertical, symbol Connector_Generic:Conn_01x06
- added J2: ~, Connector_FFC-FPC:Hirose_FH12-20S-0.5SH_1x20-1MP_P0.50mm_Horizontal, symbol PartLibrary:HS12864G19A_Elec
- added R10, R14, R15, R8: 100, Resistor_SMD:R_0603_1608Metric, symbol Device:R
- added R11, R12, R13, R3, R7, R9: 4.7R, Resistor_SMD:R_0603_1608Metric, symbol Device:R
- added R16, R4: 1M, Resistor_SMD:R_0603_1608Metric, symbol Device:R
- added R2: 10k, Resistor_SMD:R_0603_1608Metric, symbol Device:R
- added R5, R6: 0R, Resistor_SMD:R_0603_1608Metric, symbol Device:R
- added U1: STM32F030C6Tx, Package_QFP:LQFP-48_7x7mm_P0.5mm, symbol MCU_ST_STM32F0:STM32F030C6Tx
- C12, C21: footprint CAP 1206_3216 - 0.8MM -> Capacitor_SMD:C_1206_3216Metric
- C13, C14, C15, C16, C22: footprint CAP 0603_1608 -> Capacitor_SMD:C_0603_1608Metric
- R8: footprint RES 0603_1608 -> Resistor_SMD:R_0603_1608Metric
- SW1, SW2: footprint FP-FSM2JSMAA-MFG -> SamacSys_Parts:FSM2J_1
Connections:
- net 3V3: now also SW2.3, J1.6 (Pin_6), J2.11 (VDD), J2.12 (VDD), R11.1, R12.1, R13.1, R3.2, R7.1, R9.1, U1.1 (VDD), U1.24 (VDD), U1.48 (VDD), U1.9 (VDDA)
- net BTN_FWD: now also U1.25 (PB12)
- net BTN_REV: now also U1.21 (PB10)
- net BTN_STOP: now also U1.22 (PB11)
- net GND: now also C10.2, C11.2, C9.2, DSP1.2 (K), J1.3 (Pin_3), J2.13 (GND), J2.14 (GND), J2.18 (GND), J2.19 (GND), J2.MP, R16.2, R2.1, R4.2, R5.2, R6.2, U1.23 (VSS), U1.47 (VSS), U1.8 (VSSA); no longer SW2.3
- net STEPPER_DIR: now also U1.19 (PB1)
- net STEPPER_EN: now also U1.20 (PB2)
- net STEPPER_STEP: now also U1.18 (PB0)
- net EN renamed RST
- net RST: now also R14.1, U1.7 (NRST)
- net GPIO0 renamed BOOT
- net BOOT: now also R15.2, R2.2, U1.44 (BOOT0)
- new net: J1.5 (Pin_5), R8.2
- new net: C8.1, J2.15 (V0)
- new net: C8.2, J2.16 (XV0)
- new net: J1.1 (Pin_1), R14.2
- new net: J1.2 (Pin_2), R15.1
- new net: J1.4 (Pin_4), R10.2
- new net: J2.20 (ESD), R16.1
- new net: C11.1, J2.17 (VG)
- new net: DSP1.1 (A), R3.1
- new net: DSP1.MP1 (MP), R6.1
- new net: DSP1.MP2 (MP), R5.1
- new net: J2.1 (ESD), R4.1
- new net BTN_CURR: U1.45 (PB8)
- new net BTN_ENC_A: U1.28 (PB15)
- new net BTN_ENC_B: U1.27 (PB14)
- new net BTN_ENC_ENT: U1.26 (PB13)
- new net BTN_MODE: U1.46 (PB9)
- new net CURRENT_BIT1: U1.10 (PA0)
- new net CURRENT_BIT2: U1.11 (PA1)
- new net CURRENT_BIT3: U1.12 (PA2)
- new net CURRENT_BIT4: U1.13 (PA3)
- new net LCD_A0: J2.4 (A0), R11.2, U1.43 (PB7)
- new net LCD_CS: J2.2 (CS1B), R13.2, U1.41 (PB5)
- new net LCD_RST: C10.1, J2.3 (RSTB), R12.2, U1.42 (PB6)
- new net SPI1_MISO: U1.16 (PA6)
- new net SPI1_MOSI: J2.6 (SDA), R7.2, U1.17 (PA7)
- new net SPI1_NSS: U1.14 (PA4)
- new net SPI1_SCK: C9.1, J2.5 (SCL), R9.2, U1.15 (PA5)
- new net SWCLK: R10.1, U1.37 (PA14)
- new net SWDIO: R8.1, U1.34 (PA13)
- new net USART1_CK: U1.29 (PA8)
- new net USART1_CTS: U1.32 (PA11)
- new net USART1_RTS: U1.33 (PA12)
- new net USART1_RX: U1.31 (PA10)
- new net USART1_TX: U1.30 (PA9)
- no-connect marks 2 -> 10
Other:
- note added: "LCD Display"
- note removed: "OLED"
- moved on the sheet: C12, C13, C14, C15, C16, C21, C22, R8, SW1, SW2
