File: PCB/KiCAD/Buttons.kicad_sch (KiCad schematic)
At the start: 30 parts, among them SW3 C255812, SW4 C255812, SW5 C255812, SW6 C255812, SW7 C255812

Commit message: Initial PCB draft
Parts:
- removed ENC1: PEC11L-4115F-S0020, FP-PEC11L-4115F-S0020-MFG, symbol Buttons-altium-import:root_0_454af83100f22c047ab3fe85c012a7b
- added U4: EC12D1524403, SamacSys_Parts:EC12D1524403, symbol PartLibrary:EC12D1524403
- C33, C34, C35, C36, C37, C38, C39, C40: footprint CAP 0603_1608 -> Capacitor_SMD:C_0603_1608Metric
- R22, R23, R24, R25, R26, R27, R28, R29, R30, R31, R32, R33, R34, R35, R36, R37: footprint RES 0603_1608 -> Resistor_SMD:R_0603_1608Metric
- SW3, SW4, SW5, SW6, SW7: footprint FP-FSM2JSMAA-MFG -> SamacSys_Parts:FSM2J_1
Connections:
- net 3V3: now also U4.C1, U4.D1
- net GND: now also U4.MH1, U4.MH2
- net at R26.1: now also U4.A1
- net at R28.1: now also U4.E1
- net at R22.1: now also U4.B1
- net BTN_CONT renamed BTN_CURR
- net BTN_FREE renamed BTN_MODE
- net BTN_PUL_A renamed BTN_ENC_B
- net BTN_PUL_B renamed BTN_ENC_A
- net BTN_PUL_ENT renamed BTN_ENC_ENT
Other:
- moved on the sheet: C34, C36, C37, C38, C39, C40, R24, R25, R28, R29, R30, R31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

Commit message: New PCB design
Parts:
- C33, C34, C35, C36, C37, C38, C39, C40: value ${ALTIUM_VALUE} -> 100nF; symbol Buttons-altium-import:root_3_Capacitor -> Device:C; ALTIUM_VALUE 100nF -> (none); APPLICATIONS Bypass, Decoupling -> (none); CAPACITANCE 100nF -> (none); COMPONENTLINK1DESCRIPTION Datasheet -> (none); COMPONENTLINK1URL https://www.johansondielectrics.com/downloads/x2y-filter-an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 -> (none); COMPONENTLINK2DESCRIPTION DigiKey Link -> (none); COMPONENTLINK2URL https://www.digikey.com/en/products/detail/johanson-dielect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 -> (none); DEVICE PACKAGE 0603 (1608 Metric) -> (none); FEATURES Low ESL (X2Y) -> (none); LASTUPDATED 2022-05-16 11:25:57 AM -> (none); LIFECYCLE STATUS Active -> (none); MANUFACTURER Johanson Dielectrics Inc. -> (none); MINIMUM ORDER 1 -> (none); MOUNTING TYPE Surface Mount, MLCC -> (none); OPERATING TEMPERATURE -55°C ~ 125°C -> (none); PACKAGE / CASE 0603 (1608 Metric) -> (none); PACKAGING TapeAndReel -> (none); PART NUMBER 250X14W223MV4T -> (none); PART STATUS Active -> (none); PARTID 14325 -> (none); PRICE 0.07 -> (none); SERIES X2Y® -> (none); SIZE / DIMENSION 0.064" L x 0.035" W (1.63mm x 0.89mm) -> (none); SUPPLIER 1 DigiKey -> (none); SUPPLIER PART NUMBER 1 709-1087-1-ND -> (none); TEMPERATURE COEFFICIENT X7R -> (none); THICKNESS (MAX) 0.026" (0.66mm) -> (none); TOLERANCE ±20% -> (none); VOLTAGE - RATED 25V -> (none)
- R22, R24, R26, R28, R30, R32, R33, R34: value ${ALTIUM_VALUE} -> 100R; symbol Buttons-altium-import:root_0_Resistor -> Device:R; ALTIUM_VALUE 47R -> (none); COMPONENTLINK1DESCRIPTION Datasheet -> (none); COMPONENTLINK1URL https://www.seielect.com/catalog/sei-rncf.pdf -> (none); COMPONENTLINK2DESCRIPTION DigiKey Link -> (none); COMPONENTLINK2URL https://www.digikey.com/en/products/detail/stackpole-electr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 -> (none); COMPOSITION Thin Film -> (none); DEVICE PACKAGE 0603 (1608 Metric) -> (none); FEATURES Automotive AEC-Q200 -> (none); HEIGHT - SEATED (MAX) 0.022" (0.55mm) -> (none); LASTUPDATED 2022-05-20 3:01:33 PM -> (none); LIFECYCLE STATUS Active -> (none); MANUFACTURER Stackpole Electronics Inc -> (none); MINIMUM ORDER 1 -> (none); NUMBER OF TERMINATIONS 2 -> (none); OPERATING TEMPERATURE -55°C ~ 155°C -> (none); PACKAGE / CASE 0603 (1608 Metric) -> (none); PACKAGING TapeAndReel -> (none); PART NUMBER RNCF0603DTE23K2 -> (none); PART STATUS Active -> (none); PARTID 5426 -> (none); POWER (WATTS) 0.1W, 1/10W -> (none); PRICE 0.01 -> (none); RATINGS AEC-Q200 -> (none); RESISTANCE 47R -> (none); SERIES RNCF -> (none); SIZE / DIMENSION 0.061" L x 0.031" W (1.55mm x 0.80mm) -> (none); SUPPLIER 1 DigiKey -> (none); SUPPLIER DEVICE PACKAGE 0603 -> (none); SUPPLIER PART NUMBER 1 RNCF0603DTE23K2CT-ND -> (none); TEMPERATURE COEFFICIENT ±25ppm/°C -> (none); TOLERANCE ±0.5% -> (none)
- R23, R25, R27, R29, R31, R35, R36, R37: value ${ALTIUM_VALUE} -> 1k; symbol Buttons-altium-import:root_3_Resistor -> Device:R; ALTIUM_VALUE 1k -> (none); COMPONENTLINK1DESCRIPTION Datasheet -> (none); COMPONENTLINK1URL https://www.seielect.com/catalog/sei-rncf.pdf -> (none); COMPONENTLINK2DESCRIPTION DigiKey Link -> (none); COMPONENTLINK2URL https://www.digikey.com/en/products/detail/stackpole-electr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 -> (none); COMPOSITION Thin Film -> (none); DEVICE PACKAGE 0603 (1608 Metric) -> (none); FEATURES Automotive AEC-Q200 -> (none); HEIGHT - SEATED (MAX) 0.022" (0.55mm) -> (none); LASTUPDATED 2022-05-20 3:01:33 PM -> (none); LIFECYCLE STATUS Active -> (none); MANUFACTURER Stackpole Electronics Inc -> (none); MINIMUM ORDER 1 -> (none); NUMBER OF TERMINATIONS 2 -> (none); OPERATING TEMPERATURE -55°C ~ 155°C -> (none); PACKAGE / CASE 0603 (1608 Metric) -> (none); PACKAGING TapeAndReel -> (none); PART NUMBER RNCF0603DTE23K2 -> (none); PART STATUS Active -> (none); PARTID 5426 -> (none); POWER (WATTS) 0.1W, 1/10W -> (none); PRICE 0.01 -> (none); RATINGS AEC-Q200 -> (none); RESISTANCE 1k -> (none); SERIES RNCF -> (none); SIZE / DIMENSION 0.061" L x 0.031" W (1.55mm x 0.80mm) -> (none); SUPPLIER 1 DigiKey -> (none); SUPPLIER DEVICE PACKAGE 0603 -> (none); SUPPLIER PART NUMBER 1 RNCF0603DTE23K2CT-ND -> (none); TEMPERATURE COEFFICIENT ±25ppm/°C -> (none); TOLERANCE ±0.5% -> (none)

Commit message: purchased board
Parts:
- SW4: renamed from SW3; LCSC (none) -> C255812
- SW5: renamed from SW4; LCSC (none) -> C255812
- SW6: renamed from SW5; LCSC (none) -> C255812
- SW7: LCSC (none) -> C255812
- SW8: renamed from SW6; LCSC (none) -> C255812
- U4: LCSC (none) -> C112349
- renumbered C33 to C25, C34 to C26, C35 to C27, C36 to C28, C37 to C29, C38 to C30, C40 to C31, C39 to C32, R22 to R28, R23 to R29, R24 to R30, R25 to R31, R26 to R32, R27 to R33, R28 to R34, R29 to R35, R30 to R36, R31 to R37, R32 to R38, R34 to R39, R33 to R40, R35 to R41, R37 to R42, R36 to R43
