File: PCB/KiCAD/MCU.kicad_sch (KiCad schematic)
At the start: 37 parts, among them J1 Conn_01x06, SW1 C255812, SW2 C255812, U1 STM32F030C6Tx

Commit message: New PCB design
Parts:
- removed C12: ${ALTIUM_VALUE}, Capacitor_SMD:C_1206_3216Metric, symbol ESP32-altium-import:root_1_Capacitor
- removed C14: ${ALTIUM_VALUE}, Capacitor_SMD:C_0603_1608Metric, symbol ESP32-altium-import:root_3_Capacitor
- removed C16: ${ALTIUM_VALUE}, Capacitor_SMD:C_0603_1608Metric, symbol ESP32-altium-import:root_1_Capacitor
- added C1, C3, C4: 1uF, Capacitor_SMD:C_0603_1608Metric, symbol Device:C
- added C5, C6: 30pF, Capacitor_SMD:C_0603_1608Metric, symbol Device:C
- added R2: 680R, Resistor_SMD:R_0603_1608Metric, symbol Device:R
- added Y1: 8MHz, Crystal:Crystal_SMD_HC49-SD, symbol Device:Crystal
- C10: renamed from C8; symbol Device:C_Small -> Device:C
- C11: renamed from C9; symbol Device:C_Small -> Device:C
- C12: renamed from C10; symbol Device:C_Small -> Device:C
- C13: value ${ALTIUM_VALUE} -> 1uF; symbol ESP32-altium-import:root_1_Capacitor -> Device:C; ALTIUM_VALUE 1uF -> (none); APPLICATIONS Bypass, Decoupling -> (none); CAPACITANCE 1uF -> (none); COMPONENTLINK1DESCRIPTION Datasheet -> (none); COMPONENTLINK1URL https://www.johansondielectrics.com/downloads/x2y-filter-an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 -> (none); COMPONENTLINK2DESCRIPTION DigiKey Link -> (none); COMPONENTLINK2URL https://www.digikey.com/en/products/detail/johanson-dielect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 -> (none); DEVICE PACKAGE 0603 (1608 Metric) -> (none); FEATURES Low ESL (X2Y) -> (none); LASTUPDATED 2022-05-16 11:25:57 AM -> (none); LIFECYCLE STATUS Active -> (none); MANUFACTURER Johanson Dielectrics Inc. -> (none); MINIMUM ORDER 1 -> (none); MOUNTING TYPE Surface Mount, MLCC -> (none); OPERATING TEMPERATURE -55°C ~ 125°C -> (none); PACKAGE / CASE 0603 (1608 Metric) -> (none); PACKAGING TapeAndReel -> (none); PART NUMBER 250X14W223MV4T -> (none); PART STATUS Active -> (none); PARTID 14325 -> (none); PRICE 0.07 -> (none); SERIES X2Y® -> (none); SIZE / DIMENSION 0.064" L x 0.035" W (1.63mm x 0.89mm) -> (none); SUPPLIER 1 DigiKey -> (none); SUPPLIER PART NUMBER 1 709-1087-1-ND -> (none); TEMPERATURE COEFFICIENT X7R -> (none); THICKNESS (MAX) 0.026" (0.66mm) -> (none); TOLERANCE ±20% -> (none); VOLTAGE - RATED 25V -> (none)
- C13: renamed from C11; symbol Device:C_Small -> Device:C
- C15: value ${ALTIUM_VALUE} -> 100nF; symbol ESP32-altium-import:root_2_Capacitor -> Device:C; ALTIUM_VALUE 100nF -> (none); APPLICATIONS Bypass, Decoupling -> (none); CAPACITANCE 100nF -> (none); COMPONENTLINK1DESCRIPTION Datasheet -> (none); COMPONENTLINK1URL https://www.johansondielectrics.com/downloads/x2y-filter-an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 -> (none); COMPONENTLINK2DESCRIPTION DigiKey Link -> (none); COMPONENTLINK2URL https://www.digikey.com/en/products/detail/johanson-dielect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 -> (none); DEVICE PACKAGE 0603 (1608 Metric) -> (none); FEATURES Low ESL (X2Y) -> (none); LASTUPDATED 2022-05-16 11:25:57 AM -> (none); LIFECYCLE STATUS Active -> (none); MANUFACTURER Johanson Dielectrics Inc. -> (none); MINIMUM ORDER 1 -> (none); MOUNTING TYPE Surface Mount, MLCC -> (none); OPERATING TEMPERATURE -55°C ~ 125°C -> (none); PACKAGE / CASE 0603 (1608 Metric) -> (none); PACKAGING TapeAndReel -> (none); PART NUMBER 250X14W223MV4T -> (none); PART STATUS Active -> (none); PARTID 14325 -> (none); PRICE 0.07 -> (none); SERIES X2Y® -> (none); SIZE / DIMENSION 0.064" L x 0.035" W (1.63mm x 0.89mm) -> (none); SUPPLIER 1 DigiKey -> (none); SUPPLIER PART NUMBER 1 709-1087-1-ND -> (none); TEMPERATURE COEFFICIENT X7R -> (none); THICKNESS (MAX) 0.026" (0.66mm) -> (none); TOLERANCE ±20% -> (none); VOLTAGE - RATED 25V -> (none)
- C21: value ${ALTIUM_VALUE} -> 10uF; symbol ESP32-altium-import:root_1_Capacitor -> Device:C; ALTIUM_VALUE 10uF -> (none); APPLICATIONS Medical, Non-Critical -> (none); CAPACITANCE 10uF -> (none); COMPONENTLINK1DESCRIPTION Datasheet -> (none); COMPONENTLINK1URL http://datasheets.avx.com/AVX-MM.pdf -> (none); COMPONENTLINK2DESCRIPTION DigiKey Link -> (none); COMPONENTLINK2URL http://digikey.com/product-detail/en/avx-corporation/MM061A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 -> (none); DEVICE PACKAGE 1206 (3216 Metric) -> (none); LASTUPDATED 2020-09-02 1:04:46 AM -> (none); LIFECYCLE STATUS Active -> (none); MANUFACTURER AVX Corporation -> (none); MINIMUM ORDER 1 -> (none); MOUNTING TYPE Surface Mount, MLCC -> (none); OPERATING TEMPERATURE -55°C ~ 125°C -> (none); PACKAGE / CASE 1206 (3216 Metric) -> (none); PACKAGING TapeAndReel -> (none); PART NUMBER MM061A101JCT2A -> (none); PART STATUS Active -> (none); PARTID 18685 -> (none); PRICE 0.52 -> (none); SERIES MM -> (none); SIZE / DIMENSION 0.126" L x 0.063" W (3.20mm x 1.60mm) -> (none); SUPPLIER 1 DigiKey -> (none); SUPPLIER PART NUMBER 1 478-10622-1-ND -> (none); TEMPERATURE COEFFICIENT C0G, NP0 -> (none); THICKNESS (MAX) 0.029" (0.74mm) -> (none); TOLERANCE ±5% -> (none); VOLTAGE - RATED 100V -> (none)
- C22: value ${ALTIUM_VALUE} -> 100nF; symbol ESP32-altium-import:root_3_Capacitor -> Device:C; ALTIUM_VALUE 100nF -> (none); APPLICATIONS Bypass, Decoupling -> (none); CAPACITANCE 100nF -> (none); COMPONENTLINK1DESCRIPTION Datasheet -> (none); COMPONENTLINK1URL https://www.johansondielectrics.com/downloads/x2y-filter-an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 -> (none); COMPONENTLINK2DESCRIPTION DigiKey Link -> (none); COMPONENTLINK2URL https://www.digikey.com/en/products/detail/johanson-dielect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 -> (none); DEVICE PACKAGE 0603 (1608 Metric) -> (none); FEATURES Low ESL (X2Y) -> (none); LASTUPDATED 2022-05-16 11:25:57 AM -> (none); LIFECYCLE STATUS Active -> (none); MANUFACTURER Johanson Dielectrics Inc. -> (none); MINIMUM ORDER 1 -> (none); MOUNTING TYPE Surface Mount, MLCC -> (none); OPERATING TEMPERATURE -55°C ~ 125°C -> (none); PACKAGE / CASE 0603 (1608 Metric) -> (none); PACKAGING TapeAndReel -> (none); PART NUMBER 250X14W223MV4T -> (none); PART STATUS Active -> (none); PARTID 14325 -> (none); PRICE 0.07 -> (none); SERIES X2Y® -> (none); SIZE / DIMENSION 0.064" L x 0.035" W (1.63mm x 0.89mm) -> (none); SUPPLIER 1 DigiKey -> (none); SUPPLIER PART NUMBER 1 709-1087-1-ND -> (none); TEMPERATURE COEFFICIENT X7R -> (none); THICKNESS (MAX) 0.026" (0.66mm) -> (none); TOLERANCE ±20% -> (none); VOLTAGE - RATED 25V -> (none)
- J2: footprint Connector_FFC-FPC:Hirose_FH12-20S-0.5SH_1x20-1MP_P0.50mm_Horizontal -> Footprints:AFC01-S20FFC-00
- R11: renamed from R10; value 100 -> 100R
- R15: renamed from R14; value 100 -> 100R
- R16: renamed from R15; value 100 -> 100R
- R8: value ${ALTIUM_VALUE} -> 10k; symbol ESP32-altium-import:root_3_Resistor -> Device:R; ALTIUM_VALUE 10k -> (none); COMPONENTLINK1DESCRIPTION Datasheet -> (none); COMPONENTLINK1URL https://www.seielect.com/catalog/sei-rncf.pdf -> (none); COMPONENTLINK2DESCRIPTION DigiKey Link -> (none); COMPONENTLINK2URL https://www.digikey.com/en/products/detail/stackpole-electr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 -> (none); COMPOSITION Thin Film -> (none); DEVICE PACKAGE 0603 (1608 Metric) -> (none); FEATURES Automotive AEC-Q200 -> (none); HEIGHT - SEATED (MAX) 0.022" (0.55mm) -> (none); LASTUPDATED 2022-05-20 3:01:33 PM -> (none); LIFECYCLE STATUS Active -> (none); MANUFACTURER Stackpole Electronics Inc -> (none); MINIMUM ORDER 1 -> (none); NUMBER OF TERMINATIONS 2 -> (none); OPERATING TEMPERATURE -55°C ~ 155°C -> (none); PACKAGE / CASE 0603 (1608 Metric) -> (none); PACKAGING TapeAndReel -> (none); PART NUMBER RNCF0603DTE23K2 -> (none); PART STATUS Active -> (none); PARTID 5426 -> (none); POWER (WATTS) 0.1W, 1/10W -> (none); PRICE 0.01 -> (none); RATINGS AEC-Q200 -> (none); RESISTANCE 10k -> (none); SERIES RNCF -> (none); SIZE / DIMENSION 0.061" L x 0.031" W (1.55mm x 0.80mm) -> (none); SUPPLIER 1 DigiKey -> (none); SUPPLIER DEVICE PACKAGE 0603 -> (none); SUPPLIER PART NUMBER 1 RNCF0603DTE23K2CT-ND -> (none); TEMPERATURE COEFFICIENT ±25ppm/°C -> (none); TOLERANCE ±0.5% -> (none)
- R9: renamed from R8; value 100 -> 100R
- renumbered R9 to R10, R11 to R12, R12 to R13, R13 to R14, R16 to R17, R2 to R3, R3 to R4, R4 to R5, R5 to R6, R6 to R7, R7 to R8
Connections:
- net 3V3: now also C13.1, C21.1, C1.1, C3.1, C4.1; no longer C13.2, C21.2
- net GND: now also C13.2, C15.1, C21.2, C1.2, C3.2, C4.2, C5.1, C6.1; no longer C13.1, C15.2, C21.1
- net RST: now also C15.2; no longer C15.1
- net SPI1_MISO: no longer U1.16 (PA6)
- net SPI1_NSS: no longer U1.14 (PA4)
- net USART1_CK: no longer U1.29 (PA8)
- net USART1_CTS: no longer U1.32 (PA11)
- net USART1_RTS: no longer U1.33 (PA12)
- net USART1_RX: no longer U1.31 (PA10)
- net USART1_TX: no longer U1.30 (PA9)
- net STEPPER_SLEEP: now reaches U1.39 (PB3)
- net STEPPER_RST: now reaches U1.40 (PB4)
- net OSC_IN: now reaches U1.5 (PF0)
- net OSC_IN: now also C5.2, Y1.2
- net OSC_OUT: now reaches U1.6 (PF1)
- net OSC_OUT: now also R2.2
- new net: C6.2, R2.1, Y1.1
- no-connect marks 10 -> 13
Other:
- note added: "Clock"
- note added: "STM32"
- note removed: "ESP32"
- moved on the sheet: C10, C11, C12, C13, R3, R4, SW1, SW2

Commit message: purchased board
Parts:
- added TP3: SCK, TestPoint:TestPoint_Pad_D2.0mm, symbol Connector:TestPoint
- added TP4: MOSI, TestPoint:TestPoint_Pad_D2.0mm, symbol Connector:TestPoint
- DSP1, H1, H2, H3, H4: now not fitted; now left out of the parts list
- J1: LCSC (none) -> C37208
- J2: LCSC (none) -> C262274
- SW1: renamed from SW2; LCSC (none) -> C255812
- SW2: renamed from SW1; LCSC (none) -> C255812
- U1: LCSC (none) -> C62514
- Y1: LCSC (none) -> C12674
- renumbered C13 to C2, C15 to C7, C21 to C8, C22 to C9, R8 to R1
Connections:
- net SPI1_MOSI: now also TP4.1
- net SPI1_SCK: now also TP3.1
