File: PCB/KiCAD/Power.kicad_sch (KiCad schematic)
At the start: 29 parts, among them J7 USB_C_Receptacle_USB2.0_16P, U1 TPS54231DR, U2 LM317AG-TN3-R

Commit message: Initial PCB draft
Parts:
- removed C4, C5, C6: ${ALTIUM_VALUE}, CAP 0603_1608, symbol Power-altium-import:root_3_Capacitor
- removed J7: USB_C_Receptacle_USB2.0_16P, symbol Connector:USB_C_Receptacle_USB2.0_16P
- removed R3, R5: ${ALTIUM_VALUE}, RES 0603_1608, symbol Power-altium-import:root_1_Resistor
- removed R5: 10k, symbol Device:R
- removed U2: LM317AG-TN3-R, TO-252_L, symbol Power-altium-import:root_0_PM-REG-LM217M-SOT3
- added C12: ${ALTIUM_VALUE}, Capacitor_SMD:C_0603_1608Metric, symbol Power-altium-import:root_3_Capacitor
- added J3: USB_C_Receptacle_USB2.0_14P, Connector_USB:USB_C_Receptacle_GCT_USB4105-xx-A_16P_TopMnt_Horizontal, symbol Connector:USB_C_Receptacle_USB2.0_14P
- added R17: 1k, Resistor_SMD:R_0603_1608Metric, symbol Device:R
- C1, C10, C11, C9: footprint CAP 0603_1608 -> Capacitor_SMD:C_0603_1608Metric
- C2, C3, C7, C8: footprint CAP 1206_3216 - 0.8MM -> Capacitor_SMD:C_1206_3216Metric
- D1: footprint DO214AC SMA -> Diode_SMD:D_SMA
- D1: value LED -> PD OK LED; footprint (none) -> LED_SMD:LED_1206_3216Metric
- DS1: value RED LED -> 3v3 OK LED; footprint VISH-TLMS1000_V -> LED_SMD:LED_1206_3216Metric
- E1: footprint PM_5_08_90_03 -> TerminalBlock_RND:TerminalBlock_RND_205-00288_1x03_P5.08mm_Horizontal
- L1: footprint WE-PD_1050P -> SamacSys_Parts:7447714220
- R1, R2, R4, R6: footprint RES 0603_1608 -> Resistor_SMD:R_0603_1608Metric
- R18: renamed from R4; footprint (none) -> Resistor_SMD:R_0603_1608Metric
- R19: renamed from R3; footprint (none) -> Resistor_SMD:R_0603_1608Metric
- U1: footprint D0008A_L -> Package_SO:SOIC-8_3.9x4.9mm_P1.27mm
- U2: renamed from U1; value ~ -> CH224k; footprint (none) -> Package_SO:SSOP-10_3.9x4.9mm_P1.00mm
Connections:
- net +20V: now also E1.1 (A1), J3.A4 (VBUS), J3.A9 (VBUS), J3.B4 (VBUS), J3.B9 (VBUS), R17.1; no longer E1.A1
- net 3V3: now also E1.2 (A2); no longer E1.A2
- net GND: now also E1.3 (A3), C12.2, J3.A1 (GND), J3.A12 (GND), J3.B1 (GND), J3.B12 (GND), J3.S1 (SHIELD); no longer E1.A3
- net at R19.2, U2.1 (VDD): now also U2.2 (CFG2), C12.1, R17.2
- net at U2.7 (CC1): now also J3.A5 (CC1)
- net at U2.4 (DP): now also J3.A6 (D+), J3.B6 (D+)
- net at U2.5 (DM): now also J3.A7 (D-), J3.B7 (D-)
- net at U2.6 (CC2): now also J3.B5 (CC2)
- no-connect marks 4 -> 1
Other:
- note removed: "OLED Power"
- moved on the sheet: C1, C10, C11, C2, C3, C7, C8, C9, D1, DS1, L1, R1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

Commit message: New PCB design
Parts:
- removed C11: ${ALTIUM_VALUE}, Capacitor_SMD:C_0603_1608Metric, symbol Power-altium-import:root_1_Capacitor
- removed D1: PD OK LED, LED_SMD:LED_1206_3216Metric, symbol Device:LED
- removed J3: USB_C_Receptacle_USB2.0_14P, Connector_USB:USB_C_Receptacle_GCT_USB4105-xx-A_16P_TopMnt_Horizontal, symbol Connector:USB_C_Receptacle_USB2.0_14P
- removed R19: 1k, Resistor_SMD:R_0603_1608Metric, symbol Device:R
- removed R2, R4: ${ALTIUM_VALUE}, Resistor_SMD:R_0603_1608Metric, symbol Power-altium-import:root_1_Resistor
- added C22, C23, C24: 10nF, Capacitor_SMD:C_0603_1608Metric, symbol Device:C
- added J3: USB_C_PD_only, Connector_USB:USB_C_Receptacle_GCT_USB4125-xx-x_6P_TopMnt_Horizontal, symbol Connector:USB_C_Receptacle_PowerOnly_6P
- added R21, R27: 4.7k, Resistor_SMD:R_0603_1608Metric, symbol Device:R
- added R22, R23: 1k, Resistor_SMD:R_0603_1608Metric, symbol Device:R
- added R25, R26: 3k, Resistor_SMD:R_0603_1608Metric, symbol Device:R
- added SW3: PWR_SW, Footprints:Swtich SS-12F44-G5, symbol Switch:SW_SPDT
- C1: value ${ALTIUM_VALUE} -> 100nF; symbol Power-altium-import:root_2_Capacitor -> Device:C; ALTIUM_VALUE 100nF -> (none); APPLICATIONS Bypass, Decoupling -> (none); CAPACITANCE 100nF -> (none); COMPONENTLINK1DESCRIPTION Datasheet -> (none); COMPONENTLINK1URL https://www.johansondielectrics.com/downloads/x2y-filter-an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 -> (none); COMPONENTLINK2DESCRIPTION DigiKey Link -> (none); COMPONENTLINK2URL https://www.digikey.com/en/products/detail/johanson-dielect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 -> (none); DEVICE PACKAGE 0603 (1608 Metric) -> (none); FEATURES Low ESL (X2Y) -> (none); LASTUPDATED 2022-05-16 11:25:57 AM -> (none); LIFECYCLE STATUS Active -> (none); MANUFACTURER Johanson Dielectrics Inc. -> (none); MINIMUM ORDER 1 -> (none); MOUNTING TYPE Surface Mount, MLCC -> (none); OPERATING TEMPERATURE -55°C ~ 125°C -> (none); PACKAGE / CASE 0603 (1608 Metric) -> (none); PACKAGING TapeAndReel -> (none); PART NUMBER 250X14W223MV4T -> (none); PART STATUS Active -> (none); PARTID 14325 -> (none); PRICE 0.07 -> (none); SERIES X2Y® -> (none); SIZE / DIMENSION 0.064" L x 0.035" W (1.63mm x 0.89mm) -> (none); SUPPLIER 1 DigiKey -> (none); SUPPLIER PART NUMBER 1 709-1087-1-ND -> (none); TEMPERATURE COEFFICIENT X7R -> (none); THICKNESS (MAX) 0.026" (0.66mm) -> (none); TOLERANCE ±20% -> (none); VOLTAGE - RATED 25V -> (none)
- C10: value ${ALTIUM_VALUE} -> 10pF; symbol Power-altium-import:root_1_Capacitor -> Device:C; ALTIUM_VALUE 10pF -> (none); APPLICATIONS Bypass, Decoupling -> (none); CAPACITANCE 10pF -> (none); COMPONENTLINK1DESCRIPTION Datasheet -> (none); COMPONENTLINK1URL https://www.johansondielectrics.com/downloads/x2y-filter-an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 -> (none); COMPONENTLINK2DESCRIPTION DigiKey Link -> (none); COMPONENTLINK2URL https://www.digikey.com/en/products/detail/johanson-dielect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 -> (none); DEVICE PACKAGE 0603 (1608 Metric) -> (none); FEATURES Low ESL (X2Y) -> (none); LASTUPDATED 2022-05-16 11:25:57 AM -> (none); LIFECYCLE STATUS Active -> (none); MANUFACTURER Johanson Dielectrics Inc. -> (none); MINIMUM ORDER 1 -> (none); MOUNTING TYPE Surface Mount, MLCC -> (none); OPERATING TEMPERATURE -55°C ~ 125°C -> (none); PACKAGE / CASE 0603 (1608 Metric) -> (none); PACKAGING TapeAndReel -> (none); PART NUMBER 250X14W223MV4T -> (none); PART STATUS Active -> (none); PARTID 14325 -> (none); PRICE 0.07 -> (none); SERIES X2Y® -> (none); SIZE / DIMENSION 0.064" L x 0.035" W (1.63mm x 0.89mm) -> (none); SUPPLIER 1 DigiKey -> (none); SUPPLIER PART NUMBER 1 709-1087-1-ND -> (none); TEMPERATURE COEFFICIENT X7R -> (none); THICKNESS (MAX) 0.026" (0.66mm) -> (none); TOLERANCE ±20% -> (none); VOLTAGE - RATED 25V -> (none)
- C14: renamed from C12; symbol Power-altium-import:root_3_Capacitor -> Device:C
- C2, C3: value ${ALTIUM_VALUE} -> 22uF; symbol Power-altium-import:root_1_Capacitor -> Device:C; ALTIUM_VALUE 22uF -> (none); APPLICATIONS Medical, Non-Critical -> (none); CAPACITANCE 22uF -> (none); COMPONENTLINK1DESCRIPTION Datasheet -> (none); COMPONENTLINK1URL http://datasheets.avx.com/AVX-MM.pdf -> (none); COMPONENTLINK2DESCRIPTION DigiKey Link -> (none); COMPONENTLINK2URL http://digikey.com/product-detail/en/avx-corporation/MM061A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 -> (none); DEVICE PACKAGE 1206 (3216 Metric) -> (none); LASTUPDATED 2020-09-02 1:04:46 AM -> (none); LIFECYCLE STATUS Active -> (none); MANUFACTURER AVX Corporation -> (none); MINIMUM ORDER 1 -> (none); MOUNTING TYPE Surface Mount, MLCC -> (none); OPERATING TEMPERATURE -55°C ~ 125°C -> (none); PACKAGE / CASE 1206 (3216 Metric) -> (none); PACKAGING TapeAndReel -> (none); PART NUMBER MM061A101JCT2A -> (none); PART STATUS Active -> (none); PARTID 18685 -> (none); PRICE 0.52 -> (none); SERIES MM -> (none); SIZE / DIMENSION 0.126" L x 0.063" W (3.20mm x 1.60mm) -> (none); SUPPLIER 1 DigiKey -> (none); SUPPLIER PART NUMBER 1 478-10622-1-ND -> (none); TEMPERATURE COEFFICIENT C0G, NP0 -> (none); THICKNESS (MAX) 0.029" (0.74mm) -> (none); TOLERANCE ±5% -> (none); VOLTAGE - RATED 100V -> (none)
- C7, C8: value ${ALTIUM_VALUE} -> 10uF; symbol Power-altium-import:root_1_Capacitor -> Device:C; ALTIUM_VALUE 10uF -> (none); APPLICATIONS Medical, Non-Critical -> (none); CAPACITANCE 10uF -> (none); COMPONENTLINK1DESCRIPTION Datasheet -> (none); COMPONENTLINK1URL http://datasheets.avx.com/AVX-MM.pdf -> (none); COMPONENTLINK2DESCRIPTION DigiKey Link -> (none); COMPONENTLINK2URL http://digikey.com/product-detail/en/avx-corporation/MM061A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 -> (none); DEVICE PACKAGE 1206 (3216 Metric) -> (none); LASTUPDATED 2020-09-02 1:04:46 AM -> (none); LIFECYCLE STATUS Active -> (none); MANUFACTURER AVX Corporation -> (none); MINIMUM ORDER 1 -> (none); MOUNTING TYPE Surface Mount, MLCC -> (none); OPERATING TEMPERATURE -55°C ~ 125°C -> (none); PACKAGE / CASE 1206 (3216 Metric) -> (none); PACKAGING TapeAndReel -> (none); PART NUMBER MM061A101JCT2A -> (none); PART STATUS Active -> (none); PARTID 18685 -> (none); PRICE 0.52 -> (none); SERIES MM -> (none); SIZE / DIMENSION 0.126" L x 0.063" W (3.20mm x 1.60mm) -> (none); SUPPLIER 1 DigiKey -> (none); SUPPLIER PART NUMBER 1 478-10622-1-ND -> (none); TEMPERATURE COEFFICIENT C0G, NP0 -> (none); THICKNESS (MAX) 0.029" (0.74mm) -> (none); TOLERANCE ±5% -> (none); VOLTAGE - RATED 100V -> (none)
- C9: value ${ALTIUM_VALUE} -> 10nF; symbol Power-altium-import:root_1_Capacitor -> Device:C; ALTIUM_VALUE 8.2nF -> (none); APPLICATIONS Bypass, Decoupling -> (none); CAPACITANCE 8.2nF -> (none); COMPONENTLINK1DESCRIPTION Datasheet -> (none); COMPONENTLINK1URL https://www.johansondielectrics.com/downloads/x2y-filter-an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 -> (none); COMPONENTLINK2DESCRIPTION DigiKey Link -> (none); COMPONENTLINK2URL https://www.digikey.com/en/products/detail/johanson-dielect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 -> (none); DEVICE PACKAGE 0603 (1608 Metric) -> (none); FEATURES Low ESL (X2Y) -> (none); LASTUPDATED 2022-05-16 11:25:57 AM -> (none); LIFECYCLE STATUS Active -> (none); MANUFACTURER Johanson Dielectrics Inc. -> (none); MINIMUM ORDER 1 -> (none); MOUNTING TYPE Surface Mount, MLCC -> (none); OPERATING TEMPERATURE -55°C ~ 125°C -> (none); PACKAGE / CASE 0603 (1608 Metric) -> (none); PACKAGING TapeAndReel -> (none); PART NUMBER 250X14W223MV4T -> (none); PART STATUS Active -> (none); PARTID 14325 -> (none); PRICE 0.07 -> (none); SERIES X2Y® -> (none); SIZE / DIMENSION 0.064" L x 0.035" W (1.63mm x 0.89mm) -> (none); SUPPLIER 1 DigiKey -> (none); SUPPLIER PART NUMBER 1 709-1087-1-ND -> (none); TEMPERATURE COEFFICIENT X7R -> (none); THICKNESS (MAX) 0.026" (0.66mm) -> (none); TOLERANCE ±20% -> (none); VOLTAGE - RATED 25V -> (none)
- DS1: value 3v3 OK LED -> PWR LED
- E1: value Orange -> PWR OUT
- L1: footprint SamacSys_Parts:7447714220 -> Footprints:SMDRH105R
- R1: value ${ALTIUM_VALUE} -> 4.7k; symbol Power-altium-import:root_1_Resistor -> Device:R; ALTIUM_VALUE 10.2k -> (none); COMPONENTLINK1DESCRIPTION Datasheet -> (none); COMPONENTLINK1URL https://www.seielect.com/catalog/sei-rncf.pdf -> (none); COMPONENTLINK2DESCRIPTION DigiKey Link -> (none); COMPONENTLINK2URL https://www.digikey.com/en/products/detail/stackpole-electr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 -> (none); COMPOSITION Thin Film -> (none); DEVICE PACKAGE 0603 (1608 Metric) -> (none); FEATURES Automotive AEC-Q200 -> (none); HEIGHT - SEATED (MAX) 0.022" (0.55mm) -> (none); LASTUPDATED 2022-05-20 3:01:33 PM -> (none); LIFECYCLE STATUS Active -> (none); MANUFACTURER Stackpole Electronics Inc -> (none); MINIMUM ORDER 1 -> (none); NUMBER OF TERMINATIONS 2 -> (none); OPERATING TEMPERATURE -55°C ~ 155°C -> (none); PACKAGE / CASE 0603 (1608 Metric) -> (none); PACKAGING TapeAndReel -> (none); PART NUMBER RNCF0603DTE23K2 -> (none); PART STATUS Active -> (none); PARTID 5426 -> (none); POWER (WATTS) 0.1W, 1/10W -> (none); PRICE 0.01 -> (none); RATINGS AEC-Q200 -> (none); RESISTANCE 10.2k -> (none); SERIES RNCF -> (none); SIZE / DIMENSION 0.061" L x 0.031" W (1.55mm x 0.80mm) -> (none); SUPPLIER 1 DigiKey -> (none); SUPPLIER DEVICE PACKAGE 0603 -> (none); SUPPLIER PART NUMBER 1 RNCF0603DTE23K2CT-ND -> (none); TEMPERATURE COEFFICIENT ±25ppm/°C -> (none); TOLERANCE ±0.5% -> (none)
- R6: value ${ALTIUM_VALUE} -> 3k; symbol Power-altium-import:root_1_Resistor -> Device:R; ALTIUM_VALUE 3.24k -> (none); COMPONENTLINK1DESCRIPTION Datasheet -> (none); COMPONENTLINK1URL https://www.seielect.com/catalog/sei-rncf.pdf -> (none); COMPONENTLINK2DESCRIPTION DigiKey Link -> (none); COMPONENTLINK2URL https://www.digikey.com/en/products/detail/stackpole-electr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 -> (none); COMPOSITION Thin Film -> (none); DEVICE PACKAGE 0603 (1608 Metric) -> (none); FEATURES Automotive AEC-Q200 -> (none); HEIGHT - SEATED (MAX) 0.022" (0.55mm) -> (none); LASTUPDATED 2022-05-20 3:01:33 PM -> (none); LIFECYCLE STATUS Active -> (none); MANUFACTURER Stackpole Electronics Inc -> (none); MINIMUM ORDER 1 -> (none); NUMBER OF TERMINATIONS 2 -> (none); OPERATING TEMPERATURE -55°C ~ 155°C -> (none); PACKAGE / CASE 0603 (1608 Metric) -> (none); PACKAGING TapeAndReel -> (none); PART NUMBER RNCF0603DTE23K2 -> (none); PART STATUS Active -> (none); PARTID 5426 -> (none); POWER (WATTS) 0.1W, 1/10W -> (none); PRICE 0.01 -> (none); RATINGS AEC-Q200 -> (none); RESISTANCE 3.24k -> (none); SERIES RNCF -> (none); SIZE / DIMENSION 0.061" L x 0.031" W (1.55mm x 0.80mm) -> (none); SUPPLIER 1 DigiKey -> (none); SUPPLIER DEVICE PACKAGE 0603 -> (none); SUPPLIER PART NUMBER 1 RNCF0603DTE23K2CT-ND -> (none); TEMPERATURE COEFFICIENT ±25ppm/°C -> (none); TOLERANCE ±0.5% -> (none)
- U2: footprint Package_SO:SSOP-10_3.9x4.9mm_P1.00mm -> Footprints:SSOP-10_3.9x4.9mm_P1.00mm
- renumbered R17 to R18, R18 to R19
Connections:
- net +20V: now also J3.A9 (VBUS), J3.B9 (VBUS), SW3.2 (B); no longer C7.2, C8.2, U1.2 (VIN)
- net 3V3: now also C2.1, C3.1, R1.1, R22.2, R23.1; no longer C2.2, C3.2, R1.2
- net GND: now also C10.2, C2.2, C3.2, C7.2, C8.2, C9.2, R6.2, C22.2, C23.2, C24.2, J3.A12 (GND), J3.B12 (GND), J3.S1 (SHIELD); no longer C10.1, C2.1, C3.1, C7.1, C8.1, C9.1, R6.1, U2.3 (CFG3), U2.9 (CFG1)
- net at C14.1, R18.2, U2.1 (VDD): no longer U2.2 (CFG2)
- net at U1.4 (SS): now also C9.1; no longer C9.2
- net at U1.6 (COMP): now also C10.1, R25.1; no longer C10.2
- net at U2.7 (CC1): now also J3.A5 (CC1)
- net at U2.4 (DP): now also U2.5 (DM)
- net at U2.6 (CC2): now also J3.B5 (CC2)
- net at DS1.1 (A): now also R22.1, R23.2
- new net: R1.2, R21.1
- new net: C7.1, C8.1, SW3.1 (A), U1.2 (VIN)
- new net: R21.2, R6.1, U1.5 (VSENSE)
- new net: R26.2, R27.1
- new net: C22.1, C23.1, C24.1, R27.2
- new net: R25.2, R26.1
- no-connect marks 1 -> 6
Other:
- note added: "Power Indicator"
- moved on the sheet: D1, E1, L1, R18, R19, U1, U2

Commit message: purchased board
Parts:
- C14: value ${ALTIUM_VALUE} -> 1uF
- D1: LCSC (none) -> C22452
- DS1: LCSC (none) -> C84270
- J3: LCSC (none) -> C18357551
- J4: renamed from E1; LCSC (none) -> C430602
- L1: LCSC (none) -> C10165
- SW3: LCSC (none) -> C136718
- U2: LCSC (none) -> C970725
- U3: renamed from U1; LCSC (none) -> C28023
- renumbered C7 to C15, C8 to C16, C1 to C17, C2 to C18, C3 to C19, C9 to C20, C10 to C21, R1 to R20, R6 to R24
