File: PCB/KiCAD/Stepper.kicad_sch (KiCad schematic)
At the start: 15 parts, among them J4 XY115A-5.0-2P, J5 XY115A-5.0-2P, P1 22-27-2041, P2 22-27-2041, U4 TMC2209-LA

Commit message: Initial PCB draft
Parts:
- removed C30, C32: ${ALTIUM_VALUE}, CAP 0603_1608, symbol Stepper-altium-import:root_2_Capacitor
- removed C31: ${ALTIUM_VALUE}, CAP 0603_1608, symbol Stepper-altium-import:root_0_Capacitor
- removed J4, J5: XY115A-5.0-2P, 2.54-2PLTDK, symbol Stepper-altium-import:root_0_2.54-2PLTDK
- removed R20, R21: ${ALTIUM_VALUE}, RES 1206_3216, symbol Stepper-altium-import:root_0_Resistor
- removed U4: TMC2209-LA, FP-TMC2209-LA-IPC_C, symbol Stepper-altium-import:root_0_7a30eefd0264be3c54b4a2c24074cf3
- added C34, C38: 1n, Capacitor_SMD:C_0603_1608Metric, symbol Device:C
- added C35, C36, C37: 0.22u, Capacitor_SMD:C_0603_1608Metric, symbol Device:C
- added IC1: DRV8818PWPR, SamacSys_Parts:SOP65P640X120-29N, symbol PartLibrary:DRV8818PWPR
- added J4, J5: SPRING TERMINAL, Footprints:MX235-5.0-04P, symbol Connector:Screw_Terminal_01x04
- added R40, R44: 100m, Resistor_SMD:R_0603_1608Metric, symbol Device:R
- added R41, R42: 47k, Resistor_SMD:R_0603_1608Metric, symbol Device:R
- added R43: 0R, Resistor_SMD:R_0603_1608Metric, symbol Device:R
- added R45, R46: 10k, Resistor_SMD:R_0603_1608Metric, symbol Device:R
- added R47, R48, R49, R50, R51, R52, R53, R54, R55, R56, R57: 4.7k, Resistor_SMD:R_0603_1608Metric, symbol Device:R
- added TP7: DECAY, TestPoint:TestPoint_Pad_D2.0mm, symbol Connector:TestPoint
- added TP8: CURR, TestPoint:TestPoint_Pad_D2.0mm, symbol Connector:TestPoint
- C27, C28, C42: footprint CAP 0603_1608 -> Capacitor_SMD:C_0603_1608Metric
- C29, C41: footprint FP-SGV8X10_5-MFG -> Capacitor_SMD:CP_Elec_8x10
- P1, P2: footprint MOLX-22-27-2041_V -> Connector_Molex:Molex_KK-254_AE-6410-04A_1x04_P2.54mm_Vertical
Connections:
- net +20V: now also C36.2, IC1.15 (VMB), IC1.28 (VMA)
- net 3V3: now also IC1.10 (VCC), IC1.12 (USM1), IC1.13 (USM0), IC1.17 (RESETN), IC1.27 (SLEEPN), R45.2
- net GND: now also C34.1, C37.2, C38.1, IC1.21 (GND_2), IC1.29 (EP), IC1.7 (GND_1), R40.1, R41.2, R42.2, R43.1, R44.1, R46.1, R51.2
- net OA1: now also IC1.4 (AOUT1), J4.1 (Pin_1), J4.2 (Pin_2)
- net OA2: now also IC1.25 (AOUT2), J4.3 (Pin_3), J4.4 (Pin_4)
- net OB1: now also IC1.11 (BOUT1), J5.1 (Pin_1), J5.2 (Pin_2)
- net OB2: now also IC1.18 (BOUT2), J5.3 (Pin_3), J5.4 (Pin_4)
- net STEPPER_DIR: now also IC1.3 (DIR)
- net STEPPER_EN: now also IC1.26 (ENABLEN)
- net STEPPER_STEP: now also IC1.19 (STEP)
- new net: R47.2, R51.1, R52.2, R55.2
- new net: C38.2, IC1.9 (RCB), R42.1
- new net: C35.1, IC1.24 (CP2)
- new net: C35.2, IC1.23 (CP1)
- new net: C37.1, IC1.20 (VGD)
- new net: C36.1, IC1.22 (VCP)
- new net: IC1.1 (ISENA), R40.2
- new net: R49.2, R53.1, R54.2, R56.1, R57.2
- new net: R48.2, R52.1, R53.2, R55.1, R56.2
- new net: C34.2, IC1.6 (RCA), R41.1
- new net: IC1.16 (SRN), R43.2
- new net: IC1.14 (ISENB), R44.2
- new net CURRENT_BIT1: R47.1
- new net CURRENT_BIT2: R48.1
- new net CURRENT_BIT3: R49.1
- new net CURRENT_BIT4: R50.1
- new net CURRENT_SELECT: IC1.8 (VREF), R50.2, R54.1, R57.1, TP8.1
- new net DECAY_MODE: IC1.5 (DECAY), R45.1, R46.2, TP7.1
- no-connect marks 0 -> 1
Other:
- note added: "Current Configuration"
- moved on the sheet: C27, C28, C29, C41, C42, P1, P2

Commit message: New PCB design
Parts:
- removed TP7: DECAY, TestPoint:TestPoint_Pad_D2.0mm, symbol Connector:TestPoint
- added C43: 100nF, Capacitor_SMD:C_0603_1608Metric, symbol Device:C
- added R62: 4.7k, Resistor_SMD:R_0603_1608Metric, symbol Device:R
- C27, C28, C42: value ${ALTIUM_VALUE} -> 100nF; symbol Stepper-altium-import:root_3_Capacitor -> Device:C; ALTIUM_VALUE 100nF -> (none); APPLICATIONS Bypass, Decoupling -> (none); CAPACITANCE 100nF -> (none); COMPONENTLINK1DESCRIPTION Datasheet -> (none); COMPONENTLINK1URL https://www.johansondielectrics.com/downloads/x2y-filter-an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 -> (none); COMPONENTLINK2DESCRIPTION DigiKey Link -> (none); COMPONENTLINK2URL https://www.digikey.com/en/products/detail/johanson-dielect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 -> (none); DEVICE PACKAGE 0603 (1608 Metric) -> (none); FEATURES Low ESL (X2Y) -> (none); LASTUPDATED 2022-05-16 11:25:57 AM -> (none); LIFECYCLE STATUS Active -> (none); MANUFACTURER Johanson Dielectrics Inc. -> (none); MINIMUM ORDER 1 -> (none); MOUNTING TYPE Surface Mount, MLCC -> (none); OPERATING TEMPERATURE -55°C ~ 125°C -> (none); PACKAGE / CASE 0603 (1608 Metric) -> (none); PACKAGING TapeAndReel -> (none); PART NUMBER 250X14W223MV4T -> (none); PART STATUS Active -> (none); PARTID 14325 -> (none); PRICE 0.07 -> (none); SERIES X2Y® -> (none); SIZE / DIMENSION 0.064" L x 0.035" W (1.63mm x 0.89mm) -> (none); SUPPLIER 1 DigiKey -> (none); SUPPLIER PART NUMBER 1 709-1087-1-ND -> (none); TEMPERATURE COEFFICIENT X7R -> (none); THICKNESS (MAX) 0.026" (0.66mm) -> (none); TOLERANCE ±20% -> (none); VOLTAGE - RATED 25V -> (none)
- C29, C41: symbol Stepper-altium-import:root_0_203bc49f2ac43e59fd269a8c329ed05 -> Device:C_Polarized_US; CAPACITANCE 100uF -> (none); CASE/PACKAGE Radial -> (none); CONSTRUCTION Cylindrical -> (none); DIAMETER 8mm -> (none); HEIGHT 10.5mm -> (none); HEIGHT - SEATED (MAX) 0.413inch -> (none); LEAD DIAMETER 1.1mm -> (none); LEAD FREE Lead Free -> (none); LEAD PITCH 3.1mm -> (none); LEAKAGE CURRENT 3uA -> (none); LIFE (HOURS) 2000Hour -> (none); MAX OPERATING TEMPERATURE 105°C -> (none); MIN OPERATING TEMPERATURE -55°C -> (none); MOUNT Surface Mount -> (none); PACKAGE QUANTITY 500 -> (none); PACKAGING Tape and Reel -> (none); RADIATION HARDENING No -> (none); RIPPLE CURRENT 230mA -> (none); ROHS COMPLIANT Yes -> (none); SERIES SGV -> (none); TERMINATION SMD/SMT -> (none); TOLERANCE 20% -> (none); VOLTAGE 50V -> (none); VOLTAGE RATING 50V -> (none)
- C38: renamed from C34; value 1n -> 1nF
- C39: renamed from C35; value 0.22u -> 220nF
- C40: renamed from C36; value 0.22u -> 220nF
- C41: renamed from C37; value 0.22u -> 220nF
- C42: renamed from C38; value 1n -> 1nF
- R44: renamed from R40; footprint Resistor_SMD:R_0603_1608Metric -> Resistor_SMD:R_1206_3216Metric
- R48: renamed from R44; footprint Resistor_SMD:R_0603_1608Metric -> Resistor_SMD:R_1206_3216Metric
- renumbered J4 to J5, J5 to J6, R41 to R45, R42 to R46, R43 to R47, R45 to R49, R46 to R50, R47 to R51, R48 to R52, R49 to R53, R50 to R54, R51 to R55, R52 to R56, R53 to R57, R54 to R58, R55 to R59, R56 to R60, R57 to R61, TP8 to TP2
Connections:
- net +20V: now also C29.1, C41.1; no longer C29.2 (A), C41.2 (A)
- net 3V3: no longer IC1.17 (RESETN), IC1.27 (SLEEPN)
- net CURRENT_SELECT: now also R62.1
- net DECAY_MODE: now also C43.1
- net GND: now also C29.2, C41.2, C43.2, R62.2; no longer C29.1 (C), C41.1 (C)
- new net STEPPER_RST: IC1.17 (RESETN)
- new net STEPPER_SLEEP: IC1.27 (SLEEPN)
Other:
- note added: "Decay Config"
- moved on the sheet: C39, R49, R50, R51, R52, R53, R54, R55, R56, R57, R58, R59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

Commit message: purchased board
Parts:
- added TP1: STEP, TestPoint:TestPoint_Pad_D2.0mm, symbol Connector:TestPoint
- C36: renamed from C29; LCSC (none) -> C176665
- C37: renamed from C41; LCSC (none) -> C176665
- IC1: LCSC (none) -> C99045
- J5, J6: LCSC (none) -> C5349564
- P1, P2: LCSC (none) -> C239364
- TP2: now not fitted; now left out of the parts list
- renumbered C42 to C33, C27 to C34, C28 to C35
Connections:
- net STEPPER_STEP: now also TP1.1
