File: PCB/KiCAD/StepperControllerPCB.kicad_pcb (KiCad board)
At the start: 4 copper layers, 65 x 120 mm, 126 parts, among them IC1 DRV8818PWPR, J1 Conn_01x06, J3 USB_C_Receptacle_USB2.0_14P, J4 SPRING TERMINAL, J5 SPRING TERMINAL, P1 22-27-2041, P2 22-27-2041, SW1 C255812, SW2 C255812, SW3 C255812, SW4 C255812, SW5 C255812, SW6 C255812, SW7 C255812, U1 STM32F030C6Tx, U2 CH224k, U3 TPS54231DR, U4 EC12D1524403

Commit message: New PCB design
Parts:
- removed the C20 at (138.0, 79.0)
- removed the D1 at (157.5, 144.2)
- removed the R19 at (158.8, 138.8)
- removed TP7: DECAY, TestPoint:TestPoint_Pad_D2.0mm
- added C22: 10nF, Capacitor_SMD:C_0603_1608Metric, F.Cu at (140.7, 67.3)
- added C23: 10nF, Capacitor_SMD:C_0603_1608Metric, F.Cu at (139.2, 67.3)
- added C24: 10nF, Capacitor_SMD:C_0603_1608Metric, F.Cu at (137.6, 67.3)
- added C4: 1uF, Capacitor_SMD:C_0603_1608Metric, F.Cu at (126.2, 121.2)
- added C43: 100nF, Capacitor_SMD:C_0603_1608Metric, F.Cu at (159.9, 72.4)
- added C6: 30pF, Capacitor_SMD:C_0603_1608Metric, F.Cu at (129.5, 129.6)
- added R2: 680R, Resistor_SMD:R_0603_1608Metric, F.Cu at (131.5, 122.7)
- added R23: 1k, Resistor_SMD:R_0603_1608Metric, F.Cu at (122.8, 48.5)
- added R25: 3k, Resistor_SMD:R_0603_1608Metric, F.Cu at (133.4, 69.7)
- added R26: 3k, Resistor_SMD:R_0603_1608Metric, F.Cu at (136.7, 69.7)
- added R27: 4.7k, Resistor_SMD:R_0603_1608Metric, F.Cu at (139.9, 69.7)
- added R62: 4.7k, Resistor_SMD:R_0603_1608Metric, F.Cu at (169.7, 114.3)
- added SW3: PWR_SW, Footprints:Swtich SS-12F44-G5, B.Cu at (129.0, 39.7)
- added Y1: 8MHz, Crystal:Crystal_SMD_HC49-SD, F.Cu at (128.2, 126.2)
- C1: value 10uF -> 1uF; footprint Capacitor_SMD:C_1206_3216Metric -> Capacitor_SMD:C_0603_1608Metric
- C20: renamed from C18; value 8.2nF -> 10nF
- C3: value 100nF -> 1uF
- C38: renamed from C34; value 1n -> 1nF
- C39: renamed from C35; value 0.22u -> 220nF
- C40: renamed from C36; value 0.22u -> 220nF
- C41: renamed from C37; value 0.22u -> 220nF
- C42: renamed from C38; value 1n -> 1nF
- C5: value 1uF -> 30pF
- DS1: value 3v3 OK LED -> PWR LED
- J2: footprint Connector_FFC-FPC:Hirose_FH12-20S-0.5SH_1x20-1MP_P0.50mm_Horizontal -> Footprints:AFC01-S20FFC-00
- J3: value USB_C_Receptacle_USB2.0_14P -> USB_C_PD_only; footprint Connector_USB:USB_C_Receptacle_GCT_USB4105-xx-A_16P_TopMnt_Horizontal -> Connector_USB:USB_C_Receptacle_GCT_USB4125-xx-x_6P_TopMnt_Horizontal
- J4: renamed from E1; value Orange -> PWR OUT
- L1: footprint SamacSys_Parts:7447714220 -> Footprints:SMDRH105R
- R11: renamed from R10; value 100 -> 100R
- R15: renamed from R14; value 100 -> 100R
- R16: renamed from R15; value 100 -> 100R
- R20: value 10.2k -> 4.7k
- R21: value 470R -> 4.7k
- R22: value 10.5k -> 1k
- R24: renamed from R23; value 3.24k -> 3k
- R28: renamed from R24; value 47R -> 100R
- R30: renamed from R26; value 47R -> 100R
- R32: renamed from R28; value 47R -> 100R
- R34: renamed from R30; value 47R -> 100R
- R36: renamed from R32; value 47R -> 100R
- R38: renamed from R34; value 47R -> 100R
- R39: renamed from R35; value 47R -> 100R
- R40: renamed from R36; value 47R -> 100R
- R44: renamed from R40; footprint Resistor_SMD:R_0603_1608Metric -> Resistor_SMD:R_1206_3216Metric
- R48: renamed from R44; footprint Resistor_SMD:R_0603_1608Metric -> Resistor_SMD:R_1206_3216Metric
- R9: renamed from R8; value 100 -> 100R
- U2: footprint Package_SO:SSOP-10_3.9x4.9mm_P1.00mm -> Footprints:SSOP-10_3.9x4.9mm_P1.00mm
- moved R21 52.0 mm to (121.1, 84.1), turned to 180 degrees
- moved SW1 40.6 mm to (148.6, 103.4), turned to -90 degrees
- moved R22 32.8 mm to (124.2, 48.5)
- moved SW2 30.7 mm to (148.6, 110.3), turned to -90 degrees
- moved R24 21.9 mm to (121.1, 85.7), turned to 180 degrees
- moved C7 20.4 mm to (149.8, 117.2), turned to -90 degrees
- moved R1 18.9 mm to (148.2, 117.2), turned to -90 degrees
- moved R20 18.4 mm to (121.1, 82.5), turned to 0 degrees
- moved C18 17.7 mm to (120.5, 73.1), turned to -90 degrees
- moved C1 17.2 mm to (138.2, 112.1), turned to -90 degrees
- moved DS1 14.8 mm to (128.8, 48.5), turned to 0 degrees
- moved C19 13.9 mm to (123.3, 73.1), turned to -90 degrees
- moved C3 12.2 mm to (137.2, 122.2), turned to 180 degrees
- moved C21 11.8 mm to (136.0, 67.3)
- moved C16 8.65 mm to (131.5, 79.5), turned to 180 degrees
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- renumbered C8 to C10, C9 to C11, C10 to C12, C11 to C13, C12 to C14, C16 to C15, C17 to C16, C13 to C17, C14 to C18, C15 to C19, C19 to C21, C21 to C25, C22 to C26, C23 to C27, C24 to C28, C25 to C29, C26 to C30, C27 to C31, C28 to C32, C31 to C34, C32 to C35, C29 to C36, C30 to C37, C4 to C7, C6 to C8, C7 to C9, D2 to D1, J4 to J5, J5 to J6, R9 to R10, R11 to R12, R12 to R13, R13 to R14, R16 to R17, R17 to R18, R18 to R19, R25 to R29, R2 to R3, R27 to R31, R29 to R33, R31 to R35, R33 to R37, R3 to R4, R37 to R41, R38 to R42, R39 to R43, R41 to R45, R42 to R46, R43 to R47, R45 to R49, R4 to R5, R46 to R50, R47 to R51, R48 to R52, R49 to R53, R50 to R54, R51 to R55, R52 to R56, R53 to R57, R54 to R58, R55 to R59, R5 to R6, R56 to R60, R57 to R61, R6 to R7, R7 to R8, SW2 to SW1, SW1 to SW2, SW3 to SW4, SW4 to SW5, SW5 to SW6, SW6 to SW7, SW7 to SW8, TP8 to TP2
Connections:
- net /ESP32/LCD_A0 renamed /MCU/LCD_A0
- net /ESP32/LCD_CS renamed /MCU/LCD_CS
- net /ESP32/LCD_RST renamed /MCU/LCD_RST
- net /ESP32/SPI1_MOSI renamed /MCU/SPI1_MOSI
- net /ESP32/SPI1_SCK renamed /MCU/SPI1_SCK
- C1 pad 1: GND -> 3V3
- C1 pad 2: 3V3 -> GND
- C14 pad 1: Net-(U2-CFG2) -> Net-(U2-VDD)
- C15 pad 1: GND -> Net-(SW3-A)
- C15 pad 2: +20V -> GND
- C16 pad 1: GND -> Net-(SW3-A)
- C16 pad 2: +20V -> GND
- C18 pad 1: GND -> 3V3
- C18 pad 2: 3V3 -> GND
- C19 pad 1: GND -> 3V3
- C19 pad 2: 3V3 -> GND
- C2 pad 1: GND -> 3V3
- C2 pad 2: 3V3 -> GND
- C20 pad 1: GND -> Net-(U3-SS)
- C20 pad 2: Net-(U3-SS) -> GND
- C21 pad 1: GND -> Net-(U3-COMP)
- C21 pad 2: Net-(U3-COMP) -> GND
- C36 pad 1: GND -> +20V
- C36 pad 2: +20V -> GND
- C37 pad 1: GND -> +20V
- C37 pad 2: +20V -> GND
- C5 pad 2: RST -> /MCU/OSC_IN
- C7 pad 1: RST -> GND
- C7 pad 2: GND -> RST
- C8 pad 1: GND -> 3V3
- C8 pad 2: 3V3 -> GND
- IC1 pad 17: 3V3 -> STEPPER_RST
- IC1 pad 27: 3V3 -> STEPPER_SLEEP
- R18 pad 2: Net-(U2-CFG2) -> Net-(U2-VDD)
- R20 pad 1: Net-(U3-VSENSE) -> 3V3
- R20 pad 2: 3V3 -> Net-(R20-Pad2)
- R21 pad 1: Net-(DS1-A) -> Net-(R20-Pad2)
- R21 pad 2: 3V3 -> Net-(U3-VSENSE)
- R22 pad 1: Net-(C20-Pad2) -> Net-(DS1-A)
- R22 pad 2: Net-(U3-COMP) -> 3V3
- R24 pad 1: GND -> Net-(U3-VSENSE)
- R24 pad 2: Net-(U3-VSENSE) -> GND
- U1 pad 14: /ESP32/SPI1_NSS -> unconnected-(U1-PA4-Pad14)
- U1 pad 16: /ESP32/SPI1_MISO -> unconnected-(U1-PA6-Pad16)
- U1 pad 29: /ESP32/USART1_CK -> unconnected-(U1-PA8-Pad29)
- U1 pad 30: /ESP32/USART1_TX -> unconnected-(U1-PA9-Pad30)
- U1 pad 31: /ESP32/USART1_RX -> unconnected-(U1-PA10-Pad31)
- U1 pad 32: /ESP32/USART1_CTS -> unconnected-(U1-PA11-Pad32)
- U1 pad 33: /ESP32/USART1_RTS -> unconnected-(U1-PA12-Pad33)
- U1 pad 39: unconnected-(U1-PB3-Pad39) -> STEPPER_SLEEP
- U1 pad 40: unconnected-(U1-PB4-Pad40) -> STEPPER_RST
- U1 pad 5: unconnected-(U1-PF0-Pad5) -> /MCU/OSC_IN
- U1 pad 6: unconnected-(U1-PF1-Pad6) -> /MCU/OSC_OUT
- U2 pad 1: Net-(U2-CFG2) -> Net-(U2-VDD)
- U2 pad 10: Net-(D1-K) -> unconnected-(U2-PG-Pad10)
- U2 pad 2: Net-(U2-CFG2) -> unconnected-(U2-CFG2-Pad2)
- U2 pad 3: GND -> unconnected-(U2-CFG3-Pad3)
- U2 pad 4: Net-(U2-DP) -> Net-(U2-DM)
- U2 pad 9: GND -> unconnected-(U2-CFG1-Pad9)
- U3 pad 2: +20V -> Net-(SW3-A)
Routing:
- net STEPPER_SLEEP: track 0.00 -> 75.1 mm, vias 0 -> 4
- net STEPPER_RST: track 0.00 -> 73.4 mm, vias 0 -> 4
- net Net-(SW3-A): track 0.00 -> 59.8 mm, vias 0 -> 2
- net 3V3: track 108.1 -> 62.6 mm, vias 17 -> 22
- net Net-(U3-VSENSE): track 7.94 -> 34.1 mm, vias 0 -> 2
- net RST: track 51.5 -> 76.2 mm, vias 0 -> 4
- net GND: track 49.0 -> 70.3 mm, vias 62 -> 55
- net Net-(D1-K): track 19.9 -> 0.00 mm, vias 1 -> 0
- net /Stepper/DECAY_MODE: track 26.9 -> 10.7 mm, vias 2 -> 0
- net /MCU/OSC_IN: track 0.00 -> 15.3 mm
- net /Stepper/CURRENT_SELECT: track 66.2 -> 51.5 mm, vias 4 -> 3
- net BTN_CURR: track 53.5 -> 67.3 mm
- net /Stepper/OA2: track 87.2 -> 73.7 mm, vias 2 -> 5
- net Net-(U2-DP): track 11.5 -> 0.00 mm, vias 2 -> 0
- net BTN_MODE: track 51.7 -> 61.9 mm
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- added copper zone on F.Cu, net +20V
- added copper zone on F.Cu, net 3V3
- added copper zone on F.Cu, net Net-(U3-PH)
Other:
- board text added: "3v3"
- board text added: "A A B B"
- board text added: "AABB"
- board text added: "ABAB"
- board text added: "BOOT"
- board text added: "CLK"
- board text added: "CURRENT"
- board text added: "DIO"
- board text added: "GND"
- board text added: "MODE"
- board text added: "RST"
- board text added: "SETTINGS"
- board text added: "STOP"

Commit message: Added name silkscreen
Other:
- board text added: "DOMINIC PANZINO SEP 2025"
- board text added: "REV A2"

Commit message: purchased board
Parts:
- added TP1: STEP, TestPoint:TestPoint_Pad_D2.0mm, F.Cu at (164.2, 92.6)
- added TP3: SCK, TestPoint:TestPoint_Pad_D2.0mm, F.Cu at (151.7, 53.3)
- added TP4: MOSI, TestPoint:TestPoint_Pad_D2.0mm, F.Cu at (141.2, 95.4)
- moved J1 6.39 mm to (119.5, 103.6)
- moved J4 5.28 mm to (132.6, 144.8), turned to 0 degrees
- moved P2 2.57 mm to (140.9, 46.4)
- moved P1 2.57 mm to (140.9, 36.6)
- moved J5 1.50 mm to (153.0, 41.5)
- moved J3 1.35 mm to (164.8, 145.2)
- moved U4 1.00 mm to (167.0, 106.0), turned to 0 degrees
- moved J6 0.87 mm to (166.0, 41.5)
- moved SW6 0.30 mm to (166.0, 128.7)
- moved C5 0.25 mm to (126.5, 129.8)
- moved C6 0.25 mm to (129.5, 129.8)
- moved R2 0.14 mm to (131.5, 122.6)
Routing:
- net +20V: track 200.7 -> 215.5 mm
- net GND: track 70.3 -> 81.2 mm
- net /MCU/SPI1_SCK: track 77.3 -> 86.8 mm, vias 2 -> 4
- net /MCU/SPI1_MOSI: track 81.7 -> 84.2 mm
- net /Stepper/OA2: track 73.7 -> 76.1 mm
- net BTN_ENC_ENT: track 37.8 -> 39.9 mm
- net /Stepper/OB2: track 73.9 -> 76.0 mm
- net /MCU/OSC_IN: track 15.3 -> 17.4 mm
- net /Stepper/OB1: track 110.3 -> 112.3 mm
- net STEPPER_STEP: track 73.4 -> 75.3 mm
- net 3V3: track 62.6 -> 63.3 mm
Other:
- board text added: "20V"
- board text added: "REV A3"
- board text removed: "REV A2"
