File: PCB/KiCAD/StepperControllerPCB.kicad_sch (KiCad schematic)
At the start: 0 parts

Commit message: New PCB design
Other:
- sheet ESP32 renamed MCU
- sheet MCU: file ESP32.kicad_sch -> MCU.kicad_sch
Changed lines of the file:
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@@
     (stroke (width 0.1524) (type solid))
     (fill (color 0 0 0 0.0000))
-    (property "Sheetname" "ESP32" (at 20.32 15.7984 0)
+    (property "Sheetname" "MCU" (at 20.32 15.7984 0)
       (effects (font (size 1.27 1.27)) (justify left bottom))
     )
-    (property "Sheetfile" "ESP32.kicad_sch" (at 20.32 28.5246 0)
+    (property "Sheetfile" "MCU.kicad_sch" (at 20.32 28.5246 0)
       (effects (font (size 1.27 1.27)) (justify left top))
     )
